File: WeMos-RFM69.brd (EAGLE design)
At the start: 39.6 x 25.7 mm, 24 parts, among them IC1 ATSHA204A, P1 PADNORMAL, P2 PADNORMAL, P3 PADNORMAL, P4 PADNORMAL

Commit message: Version 1.0a
Parts:
- removed U$3: (no value), _c2h:LOGO_C2I_015
- added U$2: (no value), _c2h:LOGO_CH2I_75MM
- J$1: value ANTENNASMALL -> ANTENNATINY; device _c2h:SMA_UFL_PAD_SMALL -> _c2h:SMA_UFL_PAD_TINY
- moved J$1 0.20 mm to (1.97, 21.8)
Connections:
- net ANT: now also J$1.ANT3
Routing:
- net 3V3: track 81.2 -> 72.0 mm
Other:
- outline, holes or cut-outs redrawn
- board text added: "Cut Wire if you put D1 to power 1st LED with 4.3V to avoid flickering"
- board text added: "JP4"
- board text added: "V1.0a"
- board text removed: "Cut Wire if you put D1 to avoid LED pb"
- board text removed: "V1.0"
Changed lines of the file:
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@@
 <?xml version="1.0" encoding="utf-8"?>
 <!DOCTYPE eagle SYSTEM "eagle.dtd">
-<eagle version="7.5.0">
+<eagle version="7.6.0">
 <drawing>
 <settings>
@@
 <setting verticaltext="up"/>
 </settings>
-<grid distance="25" unitdist="mil" unit="mil" style="lines" multiple="1" display="yes" altdistance="5" altunitdist="mil" altunit="mil"/>
+<grid distance="25" unitdist="mil" unit="mil" style="dots" multiple="1" display="yes" altdistance="2.5" altunitdist="mil" altunit="mil"/>
 <layers>
 <layer number="1" name="Top" color="4" fill="1" visible="yes" active="yes"/>
@@
 <layer number="56" name="wert" color="7" fill="1" visible="no" active="no"/>
 <layer number="57" name="tCAD" color="7" fill="1" visible="no" active="no"/>
+<layer number="58" name="b3D" color="7" fill="1" visible="no" active="no"/>
 <layer number="59" name="tCarbon" color="7" fill="1" visible="no" active="no"/>
 <layer number="60" name="bCarbon" color="7" fill="1" visible="no" active="no"/>
@@
 <wire x1="33.655" y1="3.175" x2="33.655" y2="0" width="0.2032" layer="21"/>
 <wire x1="16.51" y1="3.81" x2="15.875" y2="3.175" width="0.2032" layer="21"/>
-<wire x1="39.97325" y1="25.527" x2="3.175" y2="25.527" width="0.0254" layer="20"/>
-<wire x1="1.778" y1="24.13" x2="1.778" y2="3.1115" width="0.0254" layer="20"/>
+<wire x1="39.97325" y1="25.527" x2="2.54" y2="25.527" width="0.0254" layer="20"/>
+<wire x1="1.778" y1="24.765" x2="1.778" y2="3.1115" width="0.0254" layer="20"/>
 <wire x1="16.4465" y1="-0.127" x2="40.0685" y2="-0.127" width="0.0254" layer="20"/>
 <wire x1="40.0685" y1="-0.127" x2="41.402" y2="1.27" width="0.0254" layer="20" curve="90"/>
@@
 <wire x1="36.83" y1="21.59" x2="38.1" y2="21.59" width="0.2032" layer="21"/>
 <text x="39.37175" y="0.51325" size="0.8128" layer="25" font="vector" ratio="15">DO</text>
-<text x="22.38375" y="18.31975" size="1.4224" layer="25" font="vector" ratio="15" align="center">RFM69
+<text x="22.00275" y="18.70075" size="1.3208" layer="25" font="vector" ratio="15" align="center">RFM69
 Gateway</text>
 <wire x1="39.37" y1="21.59" x2="40.64" y2="21.59" width="0.2032" layer="21"/>
-<wire x1="4.5593" y1="22.01545" x2="4.5593" y2="21.25345" width="0.254" layer="22" curve="69.354732"/>
-<wire x1="4.3053" y1="22.39645" x2="4.3053" y2="20.87245" width="0.254" layer="22" curve="84.805571"/>
-<wire x1="4.0513" y1="22.77745" x2="4.0513" y2="20.49145" width="0.254" layer="22" curve="90"/>
-<text x="17.93875" y="10.4775" size="1.4224" layer="26" font="vector" ratio="15" rot="MR0" align="center">V1.0</text>
+<text x="18.63725" y="10.4775" size="1.4224" layer="26" font="vector" ratio="15" rot="MR0" align="center">V1.0a</text>
 <text x="33.3375" y="7.01675" size="0.8128" layer="25" font="vector" ratio="15" rot="R90" align="center">WS2812</text>
 <wire x1="38.735" y1="0" x2="38.735" y2="3.175" width="0.2032" layer="21"/>
@@
 <wire x1="14.5415" y1="1.778" x2="3.1115" y2="1.778" width="0.0254" layer="20"/>
 <wire x1="3.1115" y1="1.778" x2="1.778" y2="3.1115" width="0.0254" layer="20" curve="-90"/>
-<wire x1="3.175" y1="25.527" x2="1.778" y2="24.13" width="0.0254" layer="20" curve="90"/>
-<text x="23.84425" y="19.1135" size="0.8128" layer="26" font="vector" ratio="15" rot="MR180" align="center">Cut Wire if you put
-D1 to avoid LED pb</text>
-<text x="12.47775" y="4.09575" size="1.4224" layer="25" font="vector" ratio="15" align="center">V1.0</text>
+<wire x1="2.54" y1="25.527" x2="1.778" y2="24.765" width="0.0254" layer="20" curve="90"/>
+<text x="22.63775" y="19.3675" size="0.8128" layer="26" font="vector" ratio="15" rot="MR180" align="center">Cut Wire if you put D1
+to power 1st LED with
+4.3V to avoid flickering</text>
+<text x="12.28725" y="23.46325" size="1.4224" layer="25" font="vector" ratio="15" align="center">V1.0a</text>
+<text x="32.22625" y="20.7645" size="0.8128" layer="26" font="vector" ratio="15" rot="MR0" align="center">JP4</text>
 </plain>
 <attributes>
@@
 <attribute name="VALUE" x="4.826" y="3.6195" size="0.8128" layer="25" font="vector" ratio="15" rot="R90"/>
 </element>
-<element name="J$1" library="_c2h" package="SMA_UFL_PAD_SMALL" value="ANTENNASMALL" x="1.905" y="21.971" rot="R180"/>
+<element name="J$1" library="_c2h" package="SMA_UFL_PAD_TINY" value="ANTENNATINY" x="1.9685" y="21.7805" rot="R180"/>
 <element name="U$4" library="_c2h" package="LOGO_CH2I_75MM" value="" x="25.2095" y="6.604" rot="MR0"/>
 <element name="BTN" library="Switch-2016" package="SW4-SMD-4.2X3.2X2.5MM" value="DHT-4235A" x="37.465" y="12.7" smashed="yes">
@@
 <attribute name="VALUE" x="10.668" y="9.906" size="0.889" layer="26" font="vector" ratio="15" rot="MR0"/>
 </element>
-<element name="U$3" library="_c2h" package="LOGO_C2I_015" value="" x="18.415" y="5.08"/>
+<element name="U$2" library="_c2h" package="LOGO_CH2I_75MM" value="" x="22.4155" y="6.985"/>
 </elements>
 <signals>
@@
 <contactref element="C4" pad="2"/>
 <contactref element="C1" pad="1"/>
-<via x="4.699" y="2.413" extent="1-16" drill="0.3556" diameter="0.7112"/>
+<via x="4.699" y="2.4765" extent="1-16" drill="0.3556" diameter="0.7112"/>
 <via x="18.288" y="7.62" extent="1-16" drill="0.3556" diameter="0.7112"/>
-<via x="22.733" y="10.414" extent="1-16" drill="0.3556" diameter="0.7112"/>
-<via x="22.225" y="16.129" extent="1-16" drill="0.3556" diameter="0.7112"/>
+<via x="22.479" y="9.906" extent="1-16" drill="0.3556" diameter="0.7112"/>
+<via x="22.4155" y="16.3195" extent="1-16" drill="0.3556" diameter="0.7112"/>
 <contactref element="U$1" pad="GND"/>
 <contactref element="U$1" pad="GND1"/>
 <via x="9.652" y="5.715" extent="1-16" drill="0.3556" diameter="0.7112"/>
 <via x="20.955" y="13.97" extent="1-16" drill="0.3556" diameter="0.7112"/>
-<via x="14.097" y="23.495" extent="1-16" drill="0.3556" diameter="0.7112"/>
+<via x="14.097" y="22.225" extent="1-16" drill="0.3556" diameter="0.7112"/>
 <contactref element="IC1" pad="4"/>
 <contactref element="C5" pad="1"/>
@@
 <contactref element="U$1" pad="SCK"/>
 <wire x1="15.495" y1="8.7" x2="24.32" y2="8.7" width="0.3048" layer="1"/>
-<wire x1="24.32" y1="8.7" x2="24.765" y2="8.255" width="0.3048" layer="1"/>
-<via x="24.765" y="8.255" extent="1-16" drill="0.3556"/>
-<wire x1="24.765" y1="8.255" x2="27.305" y2="5.715" width="0.3048" layer="16"/>
+<wire x1="24.32" y1="8.7" x2="24.511" y2="8.509" width="0.3048" layer="1"/>
+<via x="24.511" y="8.509" extent="1-16" drill="0.3556"/>
+<wire x1="24.511" y1="8.509" x2="27.305" y2="5.715" width="0.3048" layer="16"/>
 <wire x1="27.305" y1="5.715" x2="27.305" y2="1.27" width="0.3048" layer="16"/>
 <wire x1="8.51" y1="13.7" x2="9.414" y2="13.7" width="0.3048" layer="1"/>
@@
 <contactref element="U$1" pad="SDI"/>
 <wire x1="15.495" y1="10.7" x2="19.78" y2="10.7" width="0.3048" layer="1"/>
-<wire x1="19.78" y1="10.7" x2="20.447" y2="10.033" width="0.3048" layer="1"/>
-<via x="20.447" y="10.033" extent="1-16" drill="0.3556"/>
-<wire x1="20.447" y1="10.033" x2="22.225" y2="8.255" width="0.3048" layer="16"/>
+<wire x1="19.78" y1="10.7" x2="20.8915" y2="9.5885" width="0.3048" layer="1"/>
+<via x="20.8915" y="9.5885" extent="1-16" drill="0.3556"/>
+<wire x1="20.8915" y1="9.5885" x2="22.225" y2="8.255" width="0.3048" layer="16"/>
 <wire x1="22.225" y1="8.255" x2="22.225" y2="1.27" width="0.3048" layer="16"/>
 <wire x1="8.51" y1="9.7" x2="10.97" y2="9.7" width="0.3048" layer="1"/>
@@
 <contactref element="I2C_OLED" pad="1"/>
 <contactref element="C1" pad="2"/>
-<via x="19.05" y="12.954" extent="1-16" drill="0.3556" diameter="0.7112"/>
+<via x="19.05" y="13.7795" extent="1-16" drill="0.3556" diameter="0.7112"/>
 <wire x1="9.525" y1="12.97" x2="12.065" y2="12.97" width="0.6096" layer="16"/>
-<wire x1="9.525" y1="12.97" x2="17.415" y2="12.97" width="0.6096" layer="16"/>
-<wire x1="17.415" y1="12.97" x2="19.05" y2="12.954" width="0.6096" layer="16"/>
-<wire x1="12.065" y1="12.97" x2="23.13" y2="12.97" width="0.6096" layer="16"/>
+<wire x1="18.2405" y1="12.97" x2="19.05" y2="13.7795" width="0.6096" layer="16"/>
+<wire x1="12.065" y1="12.97" x2="18.2405" y2="12.97" width="0.6096" layer="16"/>
+<wire x1="18.2405" y1="12.97" x2="23.13" y2="12.97" width="0.6096" layer="16"/>
 <wire x1="23.13" y1="12.97" x2="30.5435" y2="20.3835" width="0.6096" layer="16"/>
 <wire x1="31.115" y1="20.955" x2="36.195" y2="20.955" width="0.6096" layer="16"/>
@@
 <wire x1="15.495" y1="16.7" x2="17.59" y2="16.7" width="0.6096" layer="1"/>
 <wire x1="17.59" y1="16.7" x2="19.05" y2="15.24" width="0.6096" layer="1"/>
-<wire x1="19.05" y1="15.24" x2="19.05" y2="12.954" width="0.6096" layer="1"/>
+<wire x1="19.05" y1="15.24" x2="19.05" y2="13.7795" width="0.6096" layer="1"/>
 <wire x1="28.01" y1="19.7" x2="29.86" y2="19.7" width="0.6096" layer="1"/>
 <wire x1="29.86" y1="19.7" x2="30.5435" y2="20.3835" width="0.6096" layer="1"/>
@@
 <contactref element="U$1" pad="ANT"/>
 <contactref element="U$1" pad="ANA"/>
-<wire x1="5.715" y1="21.971" x2="10.414" y2="21.971" width="0.8128" layer="1"/>
+<wire x1="6.4135" y1="21.7805" x2="10.6045" y2="21.7805" width="0.8128" layer="1"/>
 <wire x1="8.51" y1="17.7" x2="11.35" y2="17.7" width="0.8128" layer="1"/>
 <wire x1="11.35" y1="17.7" x2="12.065" y2="18.415" width="0.8128" layer="1"/>
 <wire x1="12.065" y1="18.415" x2="12.065" y2="20.32" width="0.8128" layer="1"/>
-<wire x1="12.065" y1="20.32" x2="10.414" y2="21.971" width="0.8128" layer="1"/>
+<wire x1="12.065" y1="20.32" x2="10.6045" y2="21.7805" width="0.8128" layer="1"/>
 <wire x1="15.495" y1="18.7" x2="13.685" y2="18.7" width="0.8128" layer="1"/>
 <wire x1="13.685" y1="18.7" x2="12.065" y2="20.32" width="0.8128" layer="1"/>
-<wire x1="5.715" y1="21.971" x2="4.7" y2="21.971" width="0.3048" layer="1"/>
+<wire x1="6.4135" y1="21.7805" x2="5.49375" y2="21.7805" width="0.3048" layer="1"/>
+<contactref element="J$1" pad="ANT3"/>
+<wire x1="5.23975" y1="21.7805" x2="6.4135" y2="21.7805" width="0.6096" layer="16"/>
 </signal>
 <signal name="N$1">

Commit message: Version 1.0b
OLED Display connector has now lock pad
Antenna signal with via
ground plane set to 12min blocking to avoid short circuit with
connectors
Parts:
- I2C_OLED: value CON_HEADER_1X04'SMALL'' -> CON_HEADER_1X04'LOCK'; device _c2h:M1X4 -> _c2h:1X04_LOCK
- moved I2C_OLED 5.24 mm to (5.84, 7.62)
Routing:
- net SDA: track 49.7 -> 48.7 mm
Other:
- board text added: "V1.0b"
- board text removed: "V1.0a"
